Commit message: Lidar sensor integrated on robot

File: urdf/my_robot.urdf.xacro (robot description, xacro)
@@ -6,5 +6,5 @@
   <xacro:include filename="$(find my_2wd_robot)/urdf/robot_parts/caster_wheel.urdf.xacro" />
   <xacro:include filename="$(find my_2wd_robot)/urdf/controllers/diff_drive.urdf.xacro" />
-  <xacro:include filename="$(find my_2wd_robot)/urdf/sensors/lidar_trial.xacro" />
+  <xacro:include filename="$(find my_2wd_robot)/urdf/sensors/lidar.xacro" />
   <xacro:base
     length="${base_length}"
@@ -56,58 +56,7 @@
     wheel_torque="${wheel_torque}"
   />
-  <!-- <xacro:lidar
-  radius="0.035"
-  width="0.08"
-  mass="0.1"
-  /> -->
-  <!-- Lidar sensor -->
-  <!-- <xacro:macro name="add_lidar" params="lidar_name parent_link lidar_pose">
-  <link name="${lidar_name}">
-      <visual>
-          <geometry>
-              <cylinder length="0.5" radius="0.3"/>
-          </geometry>
-          <material>
-              <color rgba="0.8784 0.6627 0.6627 1.0"/>
-          </material>
-      </visual>
-      <collision>
-          <geometry>
-              <cylinder length="0.5" radius="0.3"/>
-          </geometry>
-      </collision>
-  </link>
-  <joint name="${lidar_name}_joint" type="fixed">
-      <parent link="${parent_link}"/>
-      <child link="${lidar_name}"/>
-      <origin xyz="${lidar_pose}" rpy="0 0 0"/>
-  </joint> -->
-  <!-- Lidar plugin -->
-  <!-- <gazebo>
-      <sensor type="gpu_ray" name="${lidar_name}_sensor">
-          <pose>${lidar_pose} 0 0 0</pose>
-          <update_rate>10</update_rate>
-          <ray>
-              <scan>
-                  <horizontal>
-                      <samples>720</samples>
-                      <resolution>1</resolution>
-                      <min_angle>-1.5708</min_angle>
-                      <max_angle>1.5708</max_angle>
-                  </horizontal>
-              </scan>
-              <range>
-                  <min>0.1</min>
-                  <max>10.0</max>
-                  <resolution>0.01</resolution>
-              </range>
-          </ray>
-          <plugin name="gazebo_ros_laser_controller" filename="libgazebo_ros_gpu_laser.so">
-              <topicName>/scan</topicName>
-          </plugin>
-      </sensor>
-  </gazebo>
-</xacro:macro> -->
-<!-- Add lidar to the robot -->
-<!-- <xacro:add_lidar lidar_name="lidar" parent_link="base_link" lidar_pose="0 0 0.15"/> -->
+  <xacro:lidar
+  radius="0.05"
+  length="0.04"
+  />
 </robot>

File: urdf/sensors/lidar.xacro (robot description, xacro)
@@ -1,99 +1,70 @@
 <?xml version="1.0"?>
-<robot name="lidar" xmlns:xacro="http://ros.org/wiki/xacro">
-    <xacro:macro name="lidar" params="radius width mass">
-        <joint name="laser_joint" type="fixed">
-            <parent link="base_link"/>
-            <child link="laser_frame"/>
-            <origin xyz="0 0 0.042" rpy="0 0 0"/>
-        </joint>
-        <link name="laser_frame">
-            <visual>
-                <origin xyz="0 0 0" rpy="0 0 0"/>
-                <geometry>
-                <cylinder radius="${radius}" length="${width}"/>
-                </geometry>
-                <material name="red">
-                    <color rgba="1 0 0 1.0"/>
-                </material>
-            </visual>
-            <collision>
-                <origin xyz="0 0 0" rpy="0 0 0"/>
-                <geometry>
-                <cylinder radius="${radius}" length="${width}"/>
-                </geometry>
-            </collision>
-            <inertial>
-                <origin xyz="0 0 0" rpy="0 0 0"/>
-                <mass value="${mass}"/>
-                <inertia ixx="${(2/5) * mass * (radius * radius)}" ixy="0" ixz="0"
-                        iyy="${(2/5) * mass * (radius * radius)}" iyz="0"
-                        izz="${(2/5) * mass * (radius * radius)}" />
-            </inertial>
-        </link>
-        <gazebo reference="laser_frame">
-            <sensor name="laser" type="ray">
-                <pose>0 0 0 0 0 0</pose>
-                <always_on>true</always_on>
-                <visualize>true</visualize>
-                <update_rate>10</update_rate>
-                <ray>
-                    <scan>
-                        <horizontal>
-                            <samples>720</samples>
-                            <resolution>1</resolution>
-                            <min_angle>-3.14</min_angle>
-                            <max_angle>3.14</max_angle>
-                        </horizontal>
-                    </scan>
-                    <range>
-                        <min>0.1</min>
-                        <max>30.0</max>
-                        <resolution>0.01</resolution>
-                    </range>
-                </ray>
-                <plugin name="laser_controller" filename="gazebo_ros_ray_laser.so">
-                    <ros>
-                        <!-- <argument>~/out:=scan</argument> -->
-                        <remapping>~/out:=scan</remapping>
-                    </ros>
-                    <output_type>sensor_msgs/LaserScan</output_type>
-                    <!-- <frame_name>laser_frame</frame_name> -->
-                    <!-- <topicName>/robot/laser/scan</topicName> -->
-                </plugin>
-            </sensor>
-        </gazebo>
-        <!-- <gazebo reference="laser_frame">
-            <sensor type="gpu_ray" name="lidar">
-              <always_on>true</always_on>
-              <update_rate>10</update_rate>
-              <pose>0 0 0 0 0 0</pose>
-              <visualize>true</visualize>
-              <ray>
+<robot xmlns:xacro="http://www.ros.org/wiki/xacro" >
+    <!-- Laser inertia  -->
+    <xacro:macro name="lidar_inertial_cylinder" params="mass length radius *origin">
+        <inertial>
+            <xacro:insert_block name="origin"/>
+            <mass value="${mass}" />
+            <inertia ixx="${(1/12) * mass * (3*radius*radius + length*length)}" ixy="0.0" ixz="0.0"
+                    iyy="${(1/12) * mass * (3*radius*radius + length*length)}" iyz="0.0"
+                    izz="${(1/2) * mass * (radius*radius)}" />
+        </inertial>
+    </xacro:macro>
+    <xacro:macro name="lidar" params="radius length">
+    <!-- Laser joint  -->
+    <joint name="laser_joint" type="fixed">
+        <parent link="base_link"/>
+        <child link="laser_frame"/>
+        <origin xyz="0.1 0 0.043" rpy="0 0 0"/>
+    </joint>
+    <!-- Laser Link  -->
+    <link name="laser_frame">
+        <visual>
+            <geometry>
+                <cylinder radius="${radius}" length="${length}"/>
+            </geometry>
+            <material name="red">
+                <color rgba="1 0 0 1.0"/>
+            </material>
+        </visual>
+        <collision>
+            <geometry>
+                <cylinder radius="${radius}" length="${length}"/>
+            </geometry>
+        </collision>
+        <xacro:lidar_inertial_cylinder mass="0.1" length="${length}" radius="${radius}">
+            <origin xyz="0 0 0" rpy="0 0 0"/>
+        </xacro:lidar_inertial_cylinder>
+    </link>
+    <!-- Laser gazebo control  -->
+    <gazebo reference="laser_frame">
+        <material>Gazebo/Red</material>
+        <sensor name="laser" type="ray">
+            <pose> 0 0 0 0 0 0 </pose>
+            <visualize>true</visualize>
+            <update_rate>10</update_rate>
+            <ray>
                 <scan>
-                  <horizontal>
-                    <samples>720</samples>
-                    <resolution>1</resolution>
-                    <min_angle>-3.14</min_angle>
-                    <max_angle>3.14</max_angle>
-                  </horizontal>
+                    <horizontal>
+                        <samples>720</samples>
+                        <resolution>1</resolution>
+                        <min_angle>-3.14</min_angle>
+                        <max_angle>3.14</max_angle>
+                    </horizontal>
                 </scan>
                 <range>
-                  <min>0.1</min>
-                  <max>15.0</max>
-                  <resolution>0.01</resolution>
+                    <min>0.3</min>
+                    <max>12</max>
+                    <resolution>0.01</resolution>
                 </range>
-              </ray>
-              <plugin name="lidar_controller" filename="libgazebo_ros_gpu_sensor.so">
+            </ray>
+            <plugin name="laser_controller" filename="libgazebo_ros_ray_sensor.so">
                 <ros>
-                  <remapping>~/out:=scan</remapping>
+                    <argument>--ros-args --remap ~/out:=/scan</argument>
                 </ros>
-                <output_type>sensor_msgs/LaserScan</output_type> -->
-                <!-- <alwaysOn>true</alwaysOn> -->
-                <!-- <updateRate>10</updateRate> -->
-                <!-- <topicName>my_2wd/scan</topicName>
-                <frame_name>laser_frame</frame_name>
-              </plugin>
-            </sensor>
-        </gazebo> -->
+                <output_type>sensor_msgs/LaserScan</output_type>
+            </plugin>
+        </sensor>
+    </gazebo>
     </xacro:macro>
 </robot>
