Commit message: Spawned Multiple Robots

File: urdf/2wd_properties.urdf.xacro (robot description, xacro)
@@ -14,9 +14,3 @@
   <xacro:property name="front_caster_wheel" value="true" />
   <xacro:property name="rear_caster_wheel" value="true" />
-  <!-- <xacro:property name="laser_pose">
-    <origin xyz="0.12 0 0.33" rpy="0 0 0"/>
-  </xacro:property>
-  <xacro:property name="depth_sensor_pose">
-    <origin xyz="0.14 0.0 0.045" rpy="0 0 0"/>
-  </xacro:property> -->
 </robot>

File: urdf/my_robot.urdf.xacro (robot description, xacro)
@@ -6,5 +6,6 @@
   <xacro:include filename="$(find my_2wd_robot)/urdf/robot_parts/caster_wheel.urdf.xacro" />
   <xacro:include filename="$(find my_2wd_robot)/urdf/controllers/diff_drive.urdf.xacro" />
-  <xacro:include filename="$(find my_2wd_robot)/urdf/sensors/lidar.xacro" />
+  <!-- <xacro:include filename="$(find my_2wd_robot)/urdf/sensors/lidar.xacro" /> -->
+  <xacro:include filename="$(find my_2wd_robot)/urdf/sensors/camera.xacro" />
   <xacro:base
     length="${base_length}"
@@ -56,7 +57,11 @@
     wheel_torque="${wheel_torque}"
   />
-  <xacro:lidar
+  <!-- <xacro:lidar
   radius="0.05"
   length="0.04"
+  /> -->
+  <xacro:camera
+  radius="0.03"
+  length="0.05"
   />
 </robot>

Commit message: Update!

File: urdf/2wd_properties.urdf.xacro (robot description, xacro)
@@ -14,3 +14,5 @@
   <xacro:property name="front_caster_wheel" value="true" />
   <xacro:property name="rear_caster_wheel" value="true" />
+  <xacro:property name="lidar_enabled" value="false" />
+  <xacro:property name="camera_enabled" value="true" />
 </robot>

File: urdf/my_robot.urdf.xacro (robot description, xacro)
@@ -6,5 +6,5 @@
   <xacro:include filename="$(find my_2wd_robot)/urdf/robot_parts/caster_wheel.urdf.xacro" />
   <xacro:include filename="$(find my_2wd_robot)/urdf/controllers/diff_drive.urdf.xacro" />
-  <!-- <xacro:include filename="$(find my_2wd_robot)/urdf/sensors/lidar.xacro" /> -->
+  <xacro:include filename="$(find my_2wd_robot)/urdf/sensors/lidar.xacro" />
   <xacro:include filename="$(find my_2wd_robot)/urdf/sensors/camera.xacro" />
   <xacro:base
@@ -57,11 +57,15 @@
     wheel_torque="${wheel_torque}"
   />
-  <!-- <xacro:lidar
-  radius="0.05"
-  length="0.04"
-  /> -->
-  <xacro:camera
-  radius="0.03"
-  length="0.05"
-  />
+  <xacro:if value="${lidar_enabled}">
+    <xacro:lidar
+      radius="0.05"
+      length="0.04"
+    />
+  </xacro:if>
+  <xacro:if value="${camera_enabled}">
+    <xacro:camera
+      radius="0.03"
+      length="0.05"
+    />
+  </xacro:if>
 </robot>
